File: board/class_AB_proto_rev_1/class_AB_proto_rev_1.kicad_sch (KiCad schematic)
At the start: 4 parts, among them Q1 2N3904, Q2 2N3905

Commit message: schematic backup
Parts:
- added Q3, Q4: 2N3904, Package_TO_SOT_THT:TO-92_Inline, symbol Transistor_BJT:2N3904
- added R3: 4.7, Resistor_THT:R_Axial_DIN0207_L6.3mm_D2.5mm_P15.24mm_Horizontal, symbol Device:R_US
- added RV1: 1k, Potentiometer_SMD:Potentiometer_Bourns_3224X_Vertical, symbol Device:R_Potentiometer_US
Connections:
- net GND: now also Q4.1 (E), R3.2; no longer Q2.3 (C)
- net at Q2.2 (B): now also Q3.1 (E), RV1.3
- net at Q1.2 (B): now also Q3.3 (C), RV1.1
- new net: Q2.3 (C), Q4.2 (B), R3.1
- new net: Q3.2 (B), RV1.2
